Commit message: Add jongky_control; wire ros2_control into the URDF
diff_drive_controller 기반 컨트롤러 설정. use_mock:=true 로 하드웨어 없이
/cmd_vel -> /odom -> TF 전 경로가 돈다.

목업으로 실측 검증
- 직진 linear.x 0.2, 3초 -> odom x 0.3387 m.
  관절 10.11 rad x 반지름 0.0335 = 0.3387 로 일치
- 회전 angular.z 0.8, 3초 -> yaw +68.4도.
  관절 좌 8.04 / 우 12.18 로 갈라짐 (반시계 시 왼쪽이 덜 도는 게 정상)
- odom -> base_footprint TF 발행 확인

URDF 에 ros2_control 블록 추가. use_mock 인자로 하드웨어 플러그인을 가른다
(mock_components/GenericSystem 또는 jongky_hardware/JongkySystemHardware).
그동안 선언만 되고 미배선이던 인자에 처음으로 동작을 붙였다.

부호 반전은 URDF 나 컨트롤러 설정에 넣지 않았다. 야붐 보드는 +vx 가
물리적 후진이고 엔코더 증가도 후진인데, 그 반전은 전부 jongky_hardware
안에서 처리한다. 그래야 목업/시뮬/실물이 같은 인터페이스를 갖고
하드웨어를 갈아끼울 때 컨트롤러 설정을 안 건드린다.

설정에서 짚어둘 것
- base_frame_id 를 base_footprint 로. 기본값 base_link 를 그대로 두면
  odom 이 바퀴축 높이(33.5mm)를 기준으로 잡혀 지도가 그만큼 뜬다
- 가속 제한을 낮게 잡았다. 보드가 목표 속도까지 자체 램프를 태워서
  vx=0.15 명령에도 1.5초 시점에 0.088 m/s 밖에 못 올라간다
- update_rate 50 vs 보드 리포트 25Hz. 속도 튐은
  velocity_rolling_window_size 로 평활

Jazzy 의 diff_drive_controller 는 cmd_vel 이 TwistStamped 다 (Twist 아님).
런치에서 Command() 결과는 ParameterValue(value_type=str) 로 감싸야 한다.
둘 다 README 에 적었다.

Co-Authored-By: Claude Opus 5 <noreply@anthropic.com>

File: robot/jongky_description/urdf/jongky.urdf.xacro (robot description, xacro)
@@ -11,5 +11,5 @@
        [TBD]        센서 좌표 / 질량은 아직 추정값
        ================================================================ -->
-  <xacro:macro name="insert_robot" params="namespace is_sim:=false cam_tilt_deg laser_yaw_deg tof_pitch_deg tof_yaw_deg">
+  <xacro:macro name="insert_robot" params="namespace is_sim:=false use_mock:=false cam_tilt_deg laser_yaw_deg tof_pitch_deg tof_yaw_deg">
     <xacro:include filename="$(find jongky_description)/urdf/common/insert_inertia.urdf.xacro"/>
     <!-- ============================================================
@@ -256,4 +256,50 @@
       <origin xyz="${imu_x} 0 ${imu_z}" rpy="0 0 0"/>
     </joint>
+    <!-- ============================================================
+         ros2_control : diff_drive_controller 가 붙는 지점
+         하드웨어는 세 갈래다.
+           use_mock:=true   목업. 명령을 그대로 상태로 되돌린다.
+                            하드웨어 없이 /cmd_vel -> /odom -> TF 전 경로 검증용
+           is_sim:=true     시뮬레이터 (gz_ros2_control). 아직 미배선
+           둘 다 false      실물. jongky_hardware 플러그인
+         [부호 주의] 이 인터페이스의 관절 속도는 ROS 규약이다 —
+         양수 = 전진. 야붐 보드는 반대이므로 부호 반전은 전부
+         jongky_hardware 안에서 처리한다. 여기서는 신경 쓰지 않는다.
+         근거는 야붐보드-레퍼런스.md "부호 규약" 절.
+         ============================================================ -->
+    <ros2_control name="jongky" type="system">
+      <hardware>
+        <xacro:if value="${use_mock}">
+          <plugin>mock_components/GenericSystem</plugin>
+          <!-- 속도 명령을 적분해 위치 상태를 만들어 준다.
+               diff_drive_controller 가 position_feedback:=true 라 필요하다 -->
+          <param name="calculate_dynamics">true</param>
+        </xacro:if>
+        <xacro:unless value="${use_mock}">
+          <plugin>jongky_hardware/JongkySystemHardware</plugin>
+          <param name="serial_port">/dev/yahboom</param>
+          <param name="baud_rate">115200</param>
+          <param name="car_type">1</param>
+          <!-- [미확정] 줄자 실측으로 확정할 것 -->
+          <param name="counts_per_rev">3182</param>
+        </xacro:unless>
+      </hardware>
+      <joint name="l_wheel_joint">
+        <command_interface name="velocity">
+          <param name="min">-20.0</param>
+          <param name="max">20.0</param>
+        </command_interface>
+        <state_interface name="position"/>
+        <state_interface name="velocity"/>
+      </joint>
+      <joint name="r_wheel_joint">
+        <command_interface name="velocity">
+          <param name="min">-20.0</param>
+          <param name="max">20.0</param>
+        </command_interface>
+        <state_interface name="position"/>
+        <state_interface name="velocity"/>
+      </joint>
+    </ros2_control>
   </xacro:macro>
 </robot>

File: robot/jongky_description/urdf/robot.urdf.xacro (robot description, xacro)
@@ -9,4 +9,6 @@
   <xacro:arg name="namespace"     default=""/>
   <xacro:arg name="is_sim"        default="false"/>
+  <!-- 목업 하드웨어. 실물 없이 /cmd_vel -> /odom -> TF 를 돌려볼 때 true -->
+  <xacro:arg name="use_mock"      default="false"/>
   <xacro:arg name="cam_tilt_deg"  default="0"/>
   <!-- 라이다 스캔 0도를 로봇 정면에 맞추는 값. 실물 장착 방향에 달렸다.
@@ -27,4 +29,5 @@
   <xacro:insert_robot namespace="$(arg namespace)"
                       is_sim="$(arg is_sim)"
+                      use_mock="$(arg use_mock)"
                       cam_tilt_deg="$(arg cam_tilt_deg)"
                       laser_yaw_deg="$(arg laser_yaw_deg)"

Commit message: Add jongky_hardware: ros2_control interface for the Yahboom board
야붐 Rosmaster 보드용 SystemInterface. diff_drive_controller 가 주는
좌우 바퀴 각속도를 차체 속도로 바꿔 시리얼로 보내고, 엔코더를 관절
위치·속도로 되돌린다. 보드와 ROS 의 부호 차이를 여기서 흡수한다.

구성
- yahboom_board  : 프로토콜·시리얼·수신 스레드. ROS 를 모르고 부호도 안 다룸
- jongky_system  : ros2_control 인터페이스. 부호·단위 변환은 전부 여기
- test/fake_board.py : 보드 시뮬레이터 (pty). 하드웨어 없이 전 경로 검증

시뮬레이터로 부호 검증 완료
- ROS linear.x = +0.2 (전진)  -> 보드 vx = -0.2   (반전됨)
- ROS angular.z = +0.8 (반시계) -> 보드 vz = +0.8  (그대로)
- 엔코더 -> odom 왕복 정상

wheel_radius / wheel_separation 은 URDF 의 xacro 프로퍼티에서 직접
넘어온다. 손으로 적은 값이 형상과 어긋나는 사고를 막는다.

구현 중 잡은 것들 (README 에 상세)
- get_command(name) / set_state(name, v) 는 wait_until_set=true 로 동작해
  실시간 안전하지 않다. read()/write() 에서 쓰면 컨트롤러 매니저가 통째로
  멈춘다. 핸들을 on_activate 에서 잡고 논블로킹 오버로드를 쓰도록 수정
- last_rx_ns_ 를 open 시각으로 초기화하면 보드가 죽어 있어도 연결 성공으로
  뜬다. rx_count_ 를 따로 두어 최초 수신 여부를 구분
- 수신 프레임의 LEN 은 페이로드+3 이다. 시뮬레이터를 +2 로 만들어 1바이트
  어긋났고 프레임이 하나도 파싱되지 않았다
- pty 시험은 raw 모드 필수. 프레임 타입이 0x0A(LF)/0x0D(CR) 라 개행 변환에
  정통으로 걸린다

미완
- IMU / 배터리 토픽 발행 (파싱은 되어 있고 내보내지만 않음)
- 실물 검증. 지금까지는 시뮬레이터로만 확인

Co-Authored-By: Claude Opus 5 <noreply@anthropic.com>

File: robot/jongky_description/urdf/jongky.urdf.xacro (robot description, xacro)
@@ -11,5 +11,5 @@
        [TBD]        센서 좌표 / 질량은 아직 추정값
        ================================================================ -->
-  <xacro:macro name="insert_robot" params="namespace is_sim:=false use_mock:=false cam_tilt_deg laser_yaw_deg tof_pitch_deg tof_yaw_deg">
+  <xacro:macro name="insert_robot" params="namespace is_sim:=false use_mock:=false serial_port cam_tilt_deg laser_yaw_deg tof_pitch_deg tof_yaw_deg">
     <xacro:include filename="$(find jongky_description)/urdf/common/insert_inertia.urdf.xacro"/>
     <!-- ============================================================
@@ -278,9 +278,13 @@
         <xacro:unless value="${use_mock}">
           <plugin>jongky_hardware/JongkySystemHardware</plugin>
-          <param name="serial_port">/dev/yahboom</param>
+          <param name="serial_port">${serial_port}</param>
           <param name="baud_rate">115200</param>
           <param name="car_type">1</param>
           <!-- [미확정] 줄자 실측으로 확정할 것 -->
           <param name="counts_per_rev">3182</param>
+          <!-- 위 치수 상수를 그대로 넘긴다. 하드웨어 인터페이스가
+               바퀴속도 -> 차체속도 역산에 쓰므로 URDF 와 어긋나면 안 된다 -->
+          <param name="wheel_radius">${wheel_radius}</param>
+          <param name="wheel_separation">${wheel_y*2}</param>
         </xacro:unless>
       </hardware>

File: robot/jongky_description/urdf/robot.urdf.xacro (robot description, xacro)
@@ -11,4 +11,6 @@
   <!-- 목업 하드웨어. 실물 없이 /cmd_vel -> /odom -> TF 를 돌려볼 때 true -->
   <xacro:arg name="use_mock"      default="false"/>
+  <!-- 실물 모드에서 쓸 시리얼 포트. 가상 포트로 시험할 때 바꿔 넣는다 -->
+  <xacro:arg name="serial_port"   default="/dev/yahboom"/>
   <xacro:arg name="cam_tilt_deg"  default="0"/>
   <!-- 라이다 스캔 0도를 로봇 정면에 맞추는 값. 실물 장착 방향에 달렸다.
@@ -30,4 +32,5 @@
                       is_sim="$(arg is_sim)"
                       use_mock="$(arg use_mock)"
+                      serial_port="$(arg serial_port)"
                       cam_tilt_deg="$(arg cam_tilt_deg)"
                       laser_yaw_deg="$(arg laser_yaw_deg)"

Commit message: Calibrate wheel_separation and board PID on the real robot
제자리 회전 시험으로 트레드를 확정하고, 보드 속도 PID 의 ki 를 올렸다.
IMU 도 함께 붙여 엔코더가 못 보는 회전을 볼 수 있게 됐다.

wheel_separation 116.25 -> 119.09 mm
  5바퀴 제자리 회전 3회. 관절 변화량과 눈으로 읽은 실제 회전각으로
  역산한다.  L = r x (관절_우 - 관절_좌) / 실제회전각
    113.45 rad / 1845.0도 -> 118.03
    111.02 rad / 1782.5도 -> 119.55
    115.69 rad / 1855.0도 -> 119.71
  세 값이 1.4% 안에 모여 평균을 채택 (표준편차 0.76mm).

  [주의] odom 누적값으로 역산하면 안 된다. spin 도구는 목표에 닿는
  순간 누적을 끊지만 로봇은 감속하며 더 돈다. 눈으로 읽는 각도는 그
  감속분을 포함하므로 서로 다른 구간을 비교하게 되어 보정 부호가
  뒤집힌다. 실제로 이 실수로 116.25 -> 113.83 으로 엉뚱하게 줄였다가
  되돌렸다. 관절 변화량에는 감속분이 들어 있다.

  줄자로는 116.25 였지만(바깥면 140 / 안쪽면 92.5 / 폭 24~25) 타이어가
  눌리며 생기는 실효 트레드는 그보다 크다. 메시의 120.32 와도 가깝다.

보드 PID ki 0.06 -> 0.1
  기본값 0.06 은 약한 쪽 모터가 저속에서 데드밴드를 못 넘겨 좌우가
  5.7% 어긋난다. 0.1 로 올리면 1.6%. 0.2 까지 올리면 저속은 더 좋지만
  운용속도에서 진동이 15% -> 18% 로 늘어 두 속도의 절충점을 택했다.
  kp·kd 는 스윕해도 진동이 13~17% 에서 안 변해 공장값을 유지한다.

  URDF 파라미터로 넣어 기동할 때마다 적용한다. 보드 설정은 휘발성이라
  전원을 껐다 켜면 공장값으로 돌아간다.

캐스터 스크럽 우려는 실측으로 해소됐다. 5바퀴 제자리 회전에서
자이로/odom 비 0.99, 좌우 관절 크기차 0.3% 로 슬립 징후가 없다.

tools/jongky_calib.py
- hold: 방향 제어 직진. 차동구동은 개루프로 직진할 수 없다.
  헤딩을 되먹여 vz 로 밀면 좌우 모터가 40% 달라도 곧게 간다.
  1.9m 주행에 가로 이탈 2mm (개루프는 같은 거리에 5~6도 휨).
  PI + 데드밴드가 P 단독보다 흔들림이 27% 적다.
- spin: 관절 기준 역산으로 수정. 위 감속 구간 문제 때문이다.
- pidsweep: kp/ki/kd 중 하나를 지정해 훑는다. 목표 속도의 85% 를
  못 내는 시행은 후보에서 뺀다 (바퀴가 멈추면 진동도 0 이라 그걸
  최적으로 고르는 사고가 난다).
- 콜백을 배경 executor 스레드로 옮겼다. 제어 루프 안에서 spin_once 를
  한 번씩만 부르면 초당 150개 들어오는 메시지를 못 따라가 낡은 값으로
  제어하게 된다. 그 상태로 되먹임하면 발산한다 (헤딩 오차 RMS 29도).

알아낸 것: 좌우 진동 15~20%(3~4Hz)는 보드 PID 세 게인을 모두 훑어도
변하지 않는다. 공중에 띄워도 남는다. PID 층위가 아니라 하드웨어
(2.6kg 경량, 접지점 4개, 작은 바퀴, 엔코더 25Hz)에서 온다.
실주행 영향은 없다 — 방향 제어를 붙이면 가로 이탈 0.1% 다.

Co-Authored-By: Claude Opus 5 <noreply@anthropic.com>

File: robot/jongky_description/urdf/jongky.urdf.xacro (robot description, xacro)
@@ -21,15 +21,22 @@
          비주얼만 2.5mm 두껍게 보이고 물리·좌표에는 영향 없다. -->
     <xacro:property name="wheel_width"   value="0.0245"/>
-    <!-- wheel_y = 트레드/2 = 116.25/2
-         실측 3개가 서로 검증된다:
-            바깥면 140,  안쪽면 92.5,  바퀴 폭 24~25
-            (140 − 92.5)/2 = 23.75  ≈ 직접 잰 폭 24~25   ✓
-            트레드 = (140 + 92.5)/2 = 116.25
-         메시(wheel.stl)는 폭 27 / 트레드 120.32로 어느 것과도 안 맞는다.
-         검증된 건 base_link.stl이고 wheel.stl은 반지름 33.5 외에
-         대조된 적이 없으므로 실측을 채택한다.
-         [미확정] 최종은 제자리 회전 시험이다. 타이어가 눌리면서 생기는
-         실효 트레드는 자로 못 잰다. 1mm = 오도메트리 회전 0.9%. -->
-    <xacro:property name="wheel_y"       value="0.0581"/>
+    <!-- wheel_y = 트레드/2 = 119.09/2
+         제자리 5바퀴 회전 3회로 확정했다. 관절 변화량과 눈으로 읽은
+         실제 회전각으로 역산한다.
+           L = r x (관절_우 - 관절_좌) / 실제회전각
+           1차: 113.45 rad / 1845.0도 -> 118.03 mm
+           2차: 111.02 rad / 1782.5도 -> 119.55 mm
+           3차: 115.69 rad / 1855.0도 -> 119.71 mm
+         세 값이 1.4% 안에 모여 평균 119.09 를 쓴다 (표준편차 0.76mm).
+         [주의] odom 누적값으로 역산하면 안 된다. spin 도구는 목표에
+         닿는 순간 누적을 끊지만 로봇은 감속하며 더 돈다. 눈으로 읽는
+         각도는 그 감속분까지 포함하므로 서로 다른 구간을 비교하게 되어
+         보정 부호가 뒤집힌다. 실제로 이 실수로 116.25 -> 113.83 으로
+         엉뚱하게 줄였다가 되돌렸다. 관절 변화량에는 감속분이 들어 있다.
+         줄자로는 116.25 가 나왔지만(바깥면 140 / 안쪽면 92.5 / 폭 24~25)
+         타이어가 눌리면서 생기는 실효 트레드는 그보다 크다.
+         메시(wheel.stl)의 120.32 와도 가깝다.
+         jongky_control 의 wheel_separation 과 반드시 일치시킬 것. -->
+    <xacro:property name="wheel_y"       value="0.059545"/>
     <!-- 메시 두께 중심이 0.6mm 치우쳐 있어 보정 -->
     <xacro:property name="wheel_mesh_dy" value="0.0006"/>
@@ -293,4 +300,13 @@
                다르다. 실측 cmd 0.2 m/s -> 실제 0.144 m/s (0.719배) 이므로
                그 역수를 곱해 보낸다. 보드 가정 반지름 약 46.6mm. -->
+          <!-- 보드 속도 PID. 공장 기본은 kp 0.8 / ki 0.06 / kd 0.5 다.
+               ki 만 0.1 로 올린다 — 기본값 0.06 은 약한 쪽 모터가 저속에서
+               데드밴드를 못 넘겨 좌우가 5.7% 어긋난다. 0.1 로 올리면 1.6%.
+               더 올리면(0.2) 저속은 더 좋아지지만 운용속도에서 진동이
+               15% -> 18% 로 는다. 두 속도의 절충점이 0.1 이다.
+               측정: jongky_calib.py pidsweep, sweep 대상 ki -->
+          <param name="motor_pid_kp">0.8</param>
+          <param name="motor_pid_ki">0.1</param>
+          <param name="motor_pid_kd">0.5</param>
           <param name="board_vel_scale">1.391</param>
           <param name="wheel_radius">${wheel_radius}</param>

Commit message: Measure whether the corridor drifts instead of eyeballing it
"Does the geometry hold" was being judged by looking at seven stills, which
shows texture but not whether the corridor is still the same corridor. The data
is meant as augmentation pairs for encoder robustness, so flicker and texture
wobble are the point; a corridor that becomes a different corridor is not.

Tracks the vanishing point and the left/right wall-floor line angles across the
clip. Thresholds come from what still reads as the same hallway: 5% of frame
width is about 3 degrees at the Astra's 57.86 horizontal FOV, and 3 degrees of
wall line moves the apparent width 10cm at two metres — inside the 0.30m
inflation radius.

Also included: the five agent audits of the RL blockers, and the caster fix
they produced.

Co-Authored-By: Claude Opus 5 <noreply@anthropic.com>

File: robot/jongky_description/urdf/jongky.urdf.xacro (robot description, xacro)
@@ -46,4 +46,52 @@
     <xacro:property name="caster_y"      value="0.028"/>
     <xacro:property name="caster_z"      value="${caster_radius - wheel_radius}"/>
+    <!-- [시뮬 전용] 구르는 캐스터 (is_sim:=true 일 때만 펼쳐진다)
+         왜 필요한가 — 고정 구슬은 구르지 못하고 끌린다. 제자리 회전에서
+         구동륜과 캐스터가 같은 마찰계수를 쓰므로 비에서 mu 가 상쇄된다.
+         즉 지면 마찰을 아무리 바꿔도 이 비는 안 변한다.
+           캐스터 하중 분담 = |COM_x| / |caster_x| = 0.04942 / 0.12523 = 39.5%
+             -> N_c = 25.535 N x 0.395 = 10.08 N,  N_w = 15.46 N
+           캐스터 미끄럼 반경 r_c = sqrt(0.12523^2 + 0.028^2) = 0.12832 m
+           저항 토크 = mu x 10.08 x 0.12832 = mu x 1.2931 N.m
+           구동 토크 = mu x 15.46 x 0.059545 = mu x 0.9205 N.m
+           비 = 0.712 < 1  ->  쿨롱 기준 제자리 회전 자체가 불가능
+         실제로 Isaac 에서 최대 각속도 20초에 3.1 rad 밖에 안 돈다
+         (이론값의 1/7.4). 복도 폭을 바꿔도 같은 값이 나온다 —
+         로봇 동역학 문제이지 환경 문제가 아니다.
+         고치면 저항이 미끄럼 마찰(mu~1)에서 구름 저항(c_rr 0.01~0.05)으로
+         바뀌므로 비가 14 이상으로 올라간다.
+         (캐스터를 별도 링크로 떼면 COM 이 2.2% 뒤로 가서 미끄럼 기준 비는
+          0.712 -> 0.687 로 오히려 조금 나빠진다. 구름으로 바꾸는 것이
+          바로 그래서 유일한 답이다 — 하중 배치로는 못 뒤집는다.)
+         [이게 모델 문제라는 근거] 실물은 제자리 회전을 잘 한다. 위 wheel_y
+         를 확정한 실험 자체가 "제자리 5바퀴 회전 3회" 다. 비 0.69 가 실물의
+         물리라면 그 실험은 애초에 성립하지 않는다. 즉 0.69 는 끌리는 고정
+         구슬로 모델링한 탓이지 실물의 값이 아니다.
+         (teleop_key.py · jongky_controllers.yaml 이 말하는 "구르지 못하고
+          끌리는 고정 구슬" 은 직진 헤딩이 매번 다르게 밀린다는 관찰이다.
+          회전을 막을 정도의 저항이라는 뜻이 아니다.)
+         [안 넣은 것] 볼이 소켓 안에서 미끄러지며 생기는 저항은 모델에
+         없다. 실물 볼 캐스터면 실효 c_eff 0.1~0.2 쯤이고, 그 값이라도
+         비는 4.6~9.1 이라 회전은 문제없다. 넣고 싶으면 아래 두 관절의
+         dynamics friction 을 올리면 되는데, Isaac URDF 임포터가 그 값을
+         읽는지 확인이 안 됐고 과하게 잡으면 회전이 다시 죽는다
+         (관절당 0.05 N.m 이면 비가 0.89 로 되돌아간다). 지금은 0 으로
+         두고 tools/check_rotation.py 로 실측부터 하는 순서다.
+         [트레일] 스위블 축이 접지점보다 앞에 있어야 캐스터가 진행 방향으로
+         스스로 정렬한다. 트레일 0 이면 정렬 복원 모멘트가 없어 옆으로 그냥
+         끌리고, 고정 구슬과 다를 게 없어진다. 볼 반지름과 같은 12.5mm 를 준다.
+         스위블 각 0(직진 정렬)에서 볼 중심이 실측 캐스터 위치와 정확히
+         겹치도록 스위블 축을 caster_x + trail 에 놓는다. -->
+    <xacro:property name="caster_trail"     value="${caster_radius}"/>
+    <!-- 볼 캐스터 실물 무게. 지름 25mm 플라스틱 볼 + 요크 = 개당 20g 쯤.
+         아래에서 body_mass 에 상쇄분을 빼므로 전체 합은 2.603 kg 그대로다.
+         [주의] 0 에 가깝게 주면 안 된다. 차체와의 질량비가 커질수록 PhysX
+         관절 솔버가 흔들린다 — 바퀴(0.05kg, 50:1)가 armature 를 필요로 했던
+         것과 같은 이유다. 여기 20g 은 실물 근사이면서 비를 246:1 로 묶는다.
+         볼 관성은 2/5 m r^2 = 6.3e-7 kg.m^2 로 바퀴(2.2e-5)의 1/35 다.
+         check_rotation.py 에서 캐스터 롤 속도가 튀면 여기부터 올릴 것
+         (강철 볼이면 64g 이 실물값이고 관성도 6배가 된다). -->
+    <xacro:property name="caster_ball_mass" value="0.010"/>
+    <xacro:property name="caster_yoke_mass" value="0.010"/>
     <!-- 메시 실측 bbox (base_link.stl, mm→m 환산)
          관성 계산은 이 실제 치수로 한다. -->
@@ -98,5 +146,12 @@
             2.603 − 0.05×2 = 2.503
          바퀴 질량은 몸통의 2%라 추정 오차가 결과에 거의 영향 없다. -->
-    <xacro:property name="body_mass"     value="2.503"/>
+    <!-- is_sim 이면 캐스터를 별도 링크로 떼어내므로 그만큼 몸통에서 뺀다.
+         두 경우 모두 합계는 실측 2.603 kg 으로 같다
+         (tools/check_merged.py 가 이 합을 본다). -->
+    <xacro:property name="caster_split_mass" value="0.0"/>
+    <xacro:if value="${is_sim}">
+      <xacro:property name="caster_split_mass" value="${2*(caster_ball_mass + caster_yoke_mass)}"/>
+    </xacro:if>
+    <xacro:property name="body_mass"     value="${2.503 - caster_split_mass}"/>
     <xacro:property name="wheel_mass"    value="0.05"/>
     <xacro:property name="mesh_scale"    value="0.001 0.001 0.001"/>
@@ -137,18 +192,26 @@
         </geometry>
       </collision>
-      <!-- 왼쪽 캐스터 : 별도 링크 없이 base_link의 충돌 구슬로 처리 -->
-      <collision>
-        <origin xyz="${caster_x} ${caster_y} ${caster_z}" rpy="0 0 0"/>
-        <geometry>
-          <sphere radius="${caster_radius}"/>
-        </geometry>
-      </collision>
-      <!-- 오른쪽 캐스터 -->
-      <collision>
-        <origin xyz="${caster_x} ${-caster_y} ${caster_z}" rpy="0 0 0"/>
-        <geometry>
-          <sphere radius="${caster_radius}"/>
-        </geometry>
-      </collision>
+      <!-- 캐스터 2개 : 별도 링크 없이 base_link 의 충돌 구슬로 처리한다.
+           실물 스택은 물리를 안 돌리므로 이걸로 충분하고, 이렇게 두면
+           /joint_states 에 없는 관절이 안 생겨 robot_state_publisher 와
+           TF 가 깨끗하다.
+           시뮬(is_sim:=true)에서는 이 구슬을 빼고 아래 insert_caster 가
+           구르는 링크로 다시 세운다. 끌리는 구슬이 제자리 회전을 죽인다. -->
+      <xacro:unless value="${is_sim}">
+        <!-- 왼쪽 캐스터 -->
+        <collision>
+          <origin xyz="${caster_x} ${caster_y} ${caster_z}" rpy="0 0 0"/>
+          <geometry>
+            <sphere radius="${caster_radius}"/>
+          </geometry>
+        </collision>
+        <!-- 오른쪽 캐스터 -->
+        <collision>
+          <origin xyz="${caster_x} ${-caster_y} ${caster_z}" rpy="0 0 0"/>
+          <geometry>
+            <sphere radius="${caster_radius}"/>
+          </geometry>
+        </collision>
+      </xacro:unless>
       <!-- 관성은 콜리전 박스가 아니라 실제 차체 치수로 계산한다.
            마진 포함된 body_wid(280)를 넣으면 izz가 1.6배로 부풀어
@@ -208,4 +271,84 @@
     <xacro:insert_wheel side="l" dir="1"/>
     <xacro:insert_wheel side="r" dir="-1"/>
+    <!-- ============================================================
+         [시뮬 전용] 구르는 캐스터 — is_sim:=true 에서만 나온다
+         구조는 실물 볼 캐스터 그대로다. 관절 2개를 직렬로 건다.
+           base_link
+             └ ${side}_caster_swivel_joint  (continuous, axis Z)   요크가 방향을 튼다
+                 └ ${side}_caster_yoke
+                     └ ${side}_caster_roll_joint (continuous, axis Y)  볼이 구른다
+                         └ ${side}_caster_ball   (충돌 구슬)
+         이 두 자유도면 어느 방향으로 가도 미끄러지지 않고 구를 수 있다.
+         제자리 회전에서 캐스터가 지나가는 궤적은 반지름 0.128 m 원의
+         접선 방향(거의 ±Y)인데, 요크가 그쪽으로 돌아서면 볼은 순수 구름이
+         된다. 직진에서는 요크가 뒤로 정렬해 평범한 캐스터가 된다.
+         [왜 X·Y 두 롤 축이 아닌가] 볼 캐스터를 X롤+Y롤 짐벌로 근사하면
+         부모 X 관절이 90도 근처로 누적됐을 때 자식 Y 축이 수직이 되어
+         전진 방향 구름이 막힌다(짐벌락). 제자리 회전이 X 롤을 무한정
+         누적시키므로 반드시 그 상태를 지난다. 스위블 방식엔 그 특이점이 없다.
+         [왜 저마찰 재질(mu_caster)이 아닌가] 비가 1을 넘으려면
+         mu_c/mu_w < 0.712 이어야 한다. 그런데 PhysX 는 두 재질의 마찰을
+         기본적으로 평균으로 합치므로 캐스터 shape 을 mu=0 으로 둬도 지면
+         재질(1.0)과 평균되어 실효 0.5 밖에 안 내려간다 -> 비 1.42, 여유
+         1.4배뿐이다. 게다가 URDF 에는 접촉면별 마찰을 적을 자리가 없고
+         Isaac URDF 임포터도 로봇 전체에 재질 하나만 물린다. 즉 이 방법은
+         env 나 USD 후처리를 고쳐야 하고, 그러고도 옆으로 미는 힘 응답이
+         실물과 달라진다. 구름으로 가면 저항이 c_rr 0.01~0.05 로 떨어져
+         비가 14쯤 되고, 이건 실물 볼 캐스터의 실제 물리 그대로다.
+         [USD 변환 주의] 이 관절들은 구동하지 않는 수동 관절이다.
+         convert_urdf.py 의 joint-damping 인자는 모든 관절에 일괄로 들어간다.
+         100 으로 변환하면 캐스터가 감쇠 100 에 묶여 못 구른다 — 구동륜은
+         env 의 ImplicitActuatorCfg 가 덮어쓰지만 캐스터는 덮어쓸 주인이 없다.
+         joint-damping 을 0.0 으로 두고 변환할 것. 구동륜 게인은 어차피 env 가
+         다시 쓴다. 확인은 sim/jongky_rl/tools/check_rotation.py 가 해준다.
+         ============================================================ -->
+    <xacro:macro name="insert_caster" params="side dir">
+      <!-- 요크 : 수직축으로 도는 부분. 비주얼은 base_link.stl 이 이미
+           그리고 있으므로 넣지 않는다 (겹쳐 그리면 z-fighting 만 난다). -->
+      <link name="${side}_caster_yoke">
+        <inertial>
+          <origin xyz="${-caster_trail/2} 0 0" rpy="0 0 0"/>
+          <mass value="${caster_yoke_mass}"/>
+          <xacro:sphere_inertia m="${caster_yoke_mass}" r="${caster_radius}"/>
+        </inertial>
+      </link>
+      <!-- damping·friction 0 : 수동 관절이라 저항이 있으면 안 된다.
+           Isaac 변환기가 URDF 값을 읽는 경로로 들어올 때를 위한 명시이고,
+           CLI 인자가 이기는 경로에서는 위 [USD 변환 주의] 를 따라야 한다. -->
+      <joint name="${side}_caster_swivel_joint" type="continuous">
+        <parent link="base_link"/>
+        <child  link="${side}_caster_yoke"/>
+        <axis   xyz="0 0 1"/>
+        <origin xyz="${caster_x + caster_trail} ${dir*caster_y} ${caster_z}" rpy="0 0 0"/>
+        <dynamics damping="0.0" friction="0.0"/>
+      </joint>
+      <!-- 볼 : 접지하는 유일한 부분. 반지름은 실측 그대로 12.5mm.
+           스위블 각 0 에서 중심이 (caster_x, ±caster_y, caster_z) 에 온다 —
+           고정 구슬 시절 위치와 정확히 같다. -->
+      <link name="${side}_caster_ball">
+        <collision>
+          <origin xyz="0 0 0" rpy="0 0 0"/>
+          <geometry>
+            <sphere radius="${caster_radius}"/>
+          </geometry>
+        </collision>
+        <inertial>
+          <origin xyz="0 0 0" rpy="0 0 0"/>
+          <mass value="${caster_ball_mass}"/>
+          <xacro:sphere_inertia m="${caster_ball_mass}" r="${caster_radius}"/>
+        </inertial>
+      </link>
+      <joint name="${side}_caster_roll_joint" type="continuous">
+        <parent link="${side}_caster_yoke"/>
+        <child  link="${side}_caster_ball"/>
+        <axis   xyz="0 1 0"/>
+        <origin xyz="${-caster_trail} 0 0" rpy="0 0 0"/>
+        <dynamics damping="0.0" friction="0.0"/>
+      </joint>
+    </xacro:macro>
+    <xacro:if value="${is_sim}">
+      <xacro:insert_caster side="l" dir="1"/>
+      <xacro:insert_caster side="r" dir="-1"/>
+    </xacro:if>
     <!-- ============================================================
          센서 프레임 : 메시도 질량도 없는 빈 링크.
